Commit message: single velocity mode tested ok

File: swerve_drive_description/urdf/swerve_drive.xacro (robot description, xacro)
@@ -51,14 +51,14 @@
     </collision>
   </link>
-  <xacro:swerve_wheel side="lf"  parent="base_link">
+  <xacro:swerve_wheel side="lf_"  parent="base_link">
     <origin xyz="0.24858 0.17929 0.096509" rpy="0 0 0" />
   </xacro:swerve_wheel>
-  <xacro:swerve_wheel side="rf"  parent="base_link">
+  <xacro:swerve_wheel side="rf_"  parent="base_link">
     <origin xyz="0.24858 -0.18071 0.096509" rpy="0 0 0" />
   </xacro:swerve_wheel>
-  <xacro:swerve_wheel side="rr"  parent="base_link">
+  <xacro:swerve_wheel side="rr_"  parent="base_link">
     <origin xyz="-0.28642 -0.18071 0.096509" rpy="0 0 0" />
   </xacro:swerve_wheel>
-  <xacro:swerve_wheel side="lr"  parent="base_link">
+  <xacro:swerve_wheel side="lr_"  parent="base_link">
     <origin xyz="-0.28642 0.17929 0.096509" rpy="0 0 0" />
   </xacro:swerve_wheel>

File: swerve_drive_description/urdf/wheel.gazebo.xacro (robot description, xacro)
@@ -8,5 +8,5 @@
       <selfCollide>false</selfCollide>
     </gazebo>
-    <gazebo reference="${side}_wheel_link">
+    <gazebo reference="${side}wheel_link">
       <mu1>0.2</mu1>
       <mu2>0.2</mu2>
@@ -14,8 +14,8 @@
       <selfCollide>false</selfCollide>
     </gazebo>
-    <gazebo reference="${side}_swerve_joint">
+    <gazebo reference="${side}swerve_joint">
       <implicitSpringDamper>True</implicitSpringDamper>
     </gazebo>
-    <gazebo reference="${side}_wheel_joint">
+    <gazebo reference="${side}wheel_joint">
       <implicitSpringDamper>True</implicitSpringDamper>
     </gazebo>

File: swerve_drive_description/urdf/wheel.transmission.xacro (robot description, xacro)
@@ -4,20 +4,20 @@
   <xacro:macro name="wheel_transmission" params="side">
     <!-- all joint transmission -->
-    <transmission name="${side}_swerve_joint_trans">
+    <transmission name="${side}swerve_joint_trans">
         <type>transmission_interface/SimpleTransmission</type>
-        <joint name="${side}_swerve_joint">
+        <joint name="${side}swerve_joint">
             <hardwareInterface>hardware_interface/VelocityJointInterface</hardwareInterface>
         </joint>
-        <actuator name="${side}_swerve_joint_motor">
+        <actuator name="${side}swerve_joint_motor">
             <hardwareInterface>hardware_interface/VelocityJointInterface</hardwareInterface>
             <mechanicalReduction>1</mechanicalReduction>
         </actuator>
     </transmission>
-    <transmission name="${side}_wheel_joint_trans">
+    <transmission name="${side}wheel_joint_trans">
         <type>transmission_interface/SimpleTransmission</type>
-        <joint name="${side}_wheel_joint">
+        <joint name="${side}wheel_joint">
             <hardwareInterface>hardware_interface/VelocityJointInterface</hardwareInterface>
         </joint>
-        <actuator name="${side}_wheel_joint_motor">
+        <actuator name="${side}wheel_joint_motor">
             <hardwareInterface>hardware_interface/VelocityJointInterface</hardwareInterface>
             <mechanicalReduction>1</mechanicalReduction>

File: swerve_drive_description/urdf/wheel.xacro (robot description, xacro)
@@ -5,5 +5,5 @@
   <xacro:macro name="swerve_wheel" params="side parent *origin">
     <link
-        name="${side}_swerve_link">
+        name="${side}swerve_link">
         <inertial>
         <origin
@@ -45,5 +45,5 @@
     </link>
     <joint
-        name="${side}_swerve_joint"
+        name="${side}swerve_joint"
         type="continuous">
         <xacro:insert_block name="origin" />
@@ -51,10 +51,10 @@
         link="${parent}" />
         <child
-        link="${side}_swerve_link" />
+        link="${side}swerve_link" />
         <axis
         xyz="0 0 1" />
     </joint>
     <link
-        name="${side}_wheel_link">
+        name="${side}wheel_link">
         <inertial>
         <origin
@@ -96,5 +96,5 @@
     </link>
     <joint
-        name="${side}_wheel_joint"
+        name="${side}wheel_joint"
         type="continuous">
         <origin
@@ -102,7 +102,7 @@
         rpy="0 0 0" />
         <parent
-        link="${side}_swerve_link" />
+        link="${side}swerve_link" />
         <child
-        link="${side}_wheel_link" />
+        link="${side}wheel_link" />
         <axis
         xyz="0 -1 0" />

Commit message: load urdf param from config file

File: swerve_drive_description/urdf/swerve_drive.xacro (robot description, xacro)
@@ -1,6 +1,18 @@
 <?xml version="1.0"?>
-<robot name="swerve_drive" xmlns:xacro="http://www.ros.org/wiki/xacro">
+<robot name="$(arg name)" xmlns:xacro="http://www.ros.org/wiki/xacro">
   <xacro:include filename="$(find swerve_drive_description)/urdf/wheel.xacro" />
   <xacro:include filename="$(find swerve_drive_description)/urdf/swerve_drive.gazebo.xacro" />
+  <xacro:arg name="robot_type" default=""/>
+  <xacro:arg name="name" default="" />
+  <xacro:arg name="prefix" default="" />
+  <xacro:arg name="visual_parameters_file" default="$(find swerve_drive_description)/config/$(arg robot_type)/visual_parameters.yaml" />
+  <xacro:arg name="physical_parameters_file" default="$(find swerve_drive_description)/config/$(arg robot_type)/physical_parameters.yaml" />
+  <xacro:property name="config_visual_parameters" value="${load_yaml('$(arg visual_parameters_file)')}" />
+  <xacro:property name="config_physical_parameters" value="${load_yaml('$(arg physical_parameters_file)')}" />
+  <xacro:property name="mesh_files" value="${config_visual_parameters['mesh_files']}" />
+  <xacro:property name="joints_info" value="${config_physical_parameters['joints']}" />
+  <xacro:property name="links_info" value="${config_physical_parameters['links']}" />
+  <xacro:property name="bio" value="${links_info['base']['inertial']['origin']}" />
+  <xacro:property name="bii" value="${links_info['base']['inertial']['inertia']}" />
   <link name="base_footprint"/>
   <joint name="base_joint " type="fixed">
@@ -14,16 +26,19 @@
     name="base_link">
     <inertial>
+      <!-- <origin
+        xyz="-0.073441 0.0048344 0.14539"
+        rpy="0 0 0" /> -->
       <origin
-        xyz="-0.073441 0.0048344 0.14539"
-        rpy="0 0 0" />
+        xyz="${bio['x']} ${bio['y']} ${bio['z']}"
+        rpy="${bio['roll']} ${bio['pitch']} ${bio['yaw']}" />
       <mass
-        value="50" />
+        value="${links_info['base']['inertial']['mass']}" />
       <inertia
-        ixx="1"
+        ixx="${bii['xx']}"
         ixy="0"
         ixz="0"
-        iyy="1"
+        iyy="${bii['yy']}"
         iyz="0"
-        izz="1" />
+        izz="${bii['zz']}" />
     </inertial>
     <visual>
@@ -33,5 +48,5 @@
       <geometry>
         <mesh
-          filename="file://$(find swerve_drive_description)/meshes/base_link.STL" />
+          filename="file://$(find ${mesh_files['package']})/${mesh_files['base']['visual']['path']}" />
       </geometry>
       <material
@@ -47,19 +62,23 @@
       <geometry>
         <mesh
-          filename="file://$(find swerve_drive_description)/meshes/base_link.STL" />
+          filename="file://$(find ${mesh_files['package']})/${mesh_files['base']['collision']['path']}" />
       </geometry>
     </collision>
   </link>
-  <xacro:swerve_wheel side="lf_"  parent="base_link">
-    <origin xyz="0.24858 0.17929 0.096509" rpy="0 0 0" />
-  </xacro:swerve_wheel>
-  <xacro:swerve_wheel side="rf_"  parent="base_link">
-    <origin xyz="0.24858 -0.18071 0.096509" rpy="0 0 0" />
-  </xacro:swerve_wheel>
-  <xacro:swerve_wheel side="rr_"  parent="base_link">
-    <origin xyz="-0.28642 -0.18071 0.096509" rpy="0 0 0" />
-  </xacro:swerve_wheel>
-  <xacro:swerve_wheel side="lr_"  parent="base_link">
-    <origin xyz="-0.28642 0.17929 0.096509" rpy="0 0 0" />
-  </xacro:swerve_wheel>
+  <xacro:property name="lfj" value="${joints_info['lf']}" />
+  <xacro:property name="rfj" value="${joints_info['rf']}" />
+  <xacro:property name="rrj" value="${joints_info['rr']}" />
+  <xacro:property name="lrj" value="${joints_info['lr']}" />
+  <xacro:swerve_wheel
+    side="lf_"  parent="base_link" mesh_files="${mesh_files}" swerve_joint="${lfj}"
+    wheel_joint="${joints_info['wheel']}" links="${links_info}" />
+  <xacro:swerve_wheel
+    side="rf_"  parent="base_link" mesh_files="${mesh_files}" swerve_joint="${rfj}"
+    wheel_joint="${joints_info['wheel']}" links="${links_info}" />
+  <xacro:swerve_wheel
+    side="rr_"  parent="base_link" mesh_files="${mesh_files}" swerve_joint="${rrj}"
+    wheel_joint="${joints_info['wheel']}" links="${links_info}" />
+  <xacro:swerve_wheel
+    side="lr_"  parent="base_link" mesh_files="${mesh_files}" swerve_joint="${lrj}"
+    wheel_joint="${joints_info['wheel']}" links="${links_info}" />
 </robot>

File: swerve_drive_description/urdf/wheel.xacro (robot description, xacro)
@@ -2,43 +2,51 @@
 <robot xmlns:xacro="http://www.ros.org/wiki/xacro">
   <xacro:include filename="$(find swerve_drive_description)/urdf/wheel.gazebo.xacro" />
-  <xacro:macro name="swerve_wheel" params="side parent *origin">
+  <xacro:macro name="swerve_wheel" params="side parent  mesh_files swerve_joint wheel_joint links">
+    <xacro:property name="sjo" value="${swerve_joint['origin']}" />
+    <xacro:property name="sja" value="${swerve_joint['axis']}" />
+    <xacro:property name="wjo" value="${wheel_joint['origin']}" />
+    <xacro:property name="wja" value="${wheel_joint['axis']}" />
+    <xacro:property name="sio" value="${links['swerve']['inertial']['origin']}" />
+    <xacro:property name="sii" value="${links['swerve']['inertial']['inertia']}" />
+    <xacro:property name="wio" value="${links['wheel']['inertial']['origin']}" />
+    <xacro:property name="wii" value="${links['wheel']['inertial']['inertia']}" />
     <link
         name="${side}swerve_link">
         <inertial>
-        <origin
-            xyz="-6.5343E-06 0.003953 -0.024575"
-            rpy="0 0 0" />
-        <mass
-            value="1" />
-        <inertia
-            ixx="0.01"
-            ixy="0"
-            ixz="0"
-            iyy="0.01"
-            iyz="0"
-            izz="0.01" />
+            <origin
+                xyz="${sio['x']} ${sio['y']} ${sio['z']}"
+                rpy="${sio['roll']} ${sio['pitch']} ${sio['yaw']}" />
+            <mass
+                value="${links['swerve']['inertial']['mass']}" />
+            <inertia
+                ixx="${sii['xx']}"
+                ixy="0"
+                ixz="0"
+                iyy="${sii['yy']}"
+                iyz="0"
+                izz="${sii['zz']}" />
         </inertial>
         <visual>
-        <origin
-            xyz="0 0 0"
-            rpy="0 0 0" />
-        <geometry>
-            <mesh
-                filename="file://$(find swerve_drive_description)/meshes/swerve_link.STL" />
-        </geometry>
-        <material
-            name="">
-            <color
-            rgba="0.75294 0.75294 0.75294 1" />
-        </material>
+            <origin
+                xyz="0 0 0"
+                rpy="0 0 0" />
+            <geometry>
+                <mesh
+                    filename="file://$(find ${mesh_files['package']})/${mesh_files['swerve']['visual']['path']}" />
+            </geometry>
+            <material
+                name="">
+                <color
+                rgba="0.75294 0.75294 0.75294 1" />
+            </material>
         </visual>
         <collision>
-        <origin
-            xyz="0 0 0"
-            rpy="0 0 0" />
-        <geometry>
-            <mesh
-                filename="file://$(find swerve_drive_description)/meshes/swerve_link.STL" />
-        </geometry>
+            <origin
+                xyz="0 0 0"
+                rpy="0 0 0" />
+            <geometry>
+                <mesh
+                    filename="file://$(find ${mesh_files['package']})/${mesh_files['swerve']['collision']['path']}" />
+            </geometry>
         </collision>
     </link>
@@ -46,5 +54,7 @@
         name="${side}swerve_joint"
         type="continuous">
-        <xacro:insert_block name="origin" />
+        <origin
+            xyz="${sjo['x']} ${sjo['y']} ${sjo['z']}"
+            rpy="${sjo['roll']} ${sjo['pitch']} ${sjo['yaw']}" />
         <parent
             link="${parent}" />
@@ -52,5 +62,5 @@
             link="${side}swerve_link" />
         <axis
-            xyz="0 0 1" />
+            xyz="${sja['x']} ${sja['y']} ${sja['z']}" />
         <limit
             effort="100"
@@ -60,39 +70,39 @@
         name="${side}wheel_link">
         <inertial>
-        <origin
-            xyz="-1.1437E-05 -4.8244E-06 -7.4559E-06"
-            rpy="0 0 0" />
-        <mass
-            value="1" />
-        <inertia
-            ixx="0.01"
-            ixy="0"
-            ixz="0"
-            iyy="0.01"
-            iyz="0"
-            izz="0.01" />
+            <origin
+                xyz="${wio['x']} ${wio['y']} ${wio['z']}"
+                rpy="${wio['roll']} ${wio['pitch']} ${wio['yaw']}" />
+            <mass
+                value="${links['swerve']['inertial']['mass']}" />
+            <inertia
+                ixx="${wii['xx']}"
+                ixy="0"
+                ixz="0"
+                iyy="${wii['yy']}"
+                iyz="0"
+                izz="${wii['zz']}" />
         </inertial>
         <visual>
-        <origin
-            xyz="0 0 0"
-            rpy="0 0 0" />
-        <geometry>
-            <mesh
-                filename="file://$(find swerve_drive_description)/meshes/wheel_link.STL" />
-        </geometry>
-        <material
-            name="">
-            <color
-            rgba="0.75294 0.75294 0.75294 1" />
-        </material>
+            <origin
+                xyz="0 0 0"
+                rpy="0 0 0" />
+            <geometry>
+                <mesh
+                    filename="file://$(find ${mesh_files['package']})/${mesh_files['wheel']['visual']['path']}" />
+            </geometry>
+            <material
+                name="">
+                <color
+                rgba="0.75294 0.75294 0.75294 1" />
+            </material>
         </visual>
         <collision>
-        <origin
-            xyz="0 0 0"
-            rpy="0 0 0" />
-        <geometry>
-            <mesh
-                filename="file://$(find swerve_drive_description)/meshes/wheel_link.STL" />
-        </geometry>
+            <origin
+                xyz="0 0 0"
+                rpy="0 0 0" />
+            <geometry>
+                <mesh
+                    filename="file://$(find ${mesh_files['package']})/${mesh_files['wheel']['collision']['path']}" />
+            </geometry>
         </collision>
     </link>
@@ -101,6 +111,6 @@
         type="continuous">
         <origin
-            xyz="0 0.00047482 -0.07"
-            rpy="0 0 0" />
+            xyz="${wjo['x']} ${wjo['y']} ${wjo['z']}"
+            rpy="${wjo['roll']} ${wjo['pitch']} ${wjo['yaw']}" />
         <parent
             link="${side}swerve_link" />
@@ -108,5 +118,5 @@
             link="${side}wheel_link" />
         <axis
-            xyz="0 1 0" />
+            xyz="${wja['x']} ${wja['y']} ${wja['z']}" />
         <limit
             effort="0.3"

Commit message: setup yhs_fw01's parameters

File: swerve_drive_description/urdf/swerve_drive.xacro (robot description, xacro)
@@ -15,9 +15,10 @@
   <xacro:property name="bio" value="${links_info['base']['inertial']['origin']}" />
   <xacro:property name="bii" value="${links_info['base']['inertial']['inertia']}" />
+  <xacro:property name="jbo" value="${joints_info['base']['origin']}" />
   <link name="base_footprint"/>
   <joint name="base_joint " type="fixed">
     <origin
-      xyz="0 0 0.0485"
-      rpy="0 0 0" />
+      xyz="${jbo['x']} ${jbo['y']} ${jbo['z']}"
+      rpy="${jbo['roll']} ${jbo['pitch']} ${jbo['yaw']}" />
     <parent link="base_footprint"/>
     <child link="base_link"/>
@@ -26,7 +27,4 @@
     name="base_link">
     <inertial>
-      <!-- <origin
-        xyz="-0.073441 0.0048344 0.14539"
-        rpy="0 0 0" /> -->
       <origin
         xyz="${bio['x']} ${bio['y']} ${bio['z']}"
