Commit message: controller manager loading ok

File: swerve_drive_description/urdf/swerve_drive.gazebo.xacro (robot description, xacro)
@@ -1,4 +1,5 @@
 <?xml version="1.0"?>
 <robot name="swerve_drive" xmlns:xacro="http://www.ros.org/wiki/xacro">
+  <xacro:include filename="$(find swerve_drive_description)/urdf/wheel.transmission.xacro" />
   <physics type='ode'>
     <max_step_size>0.001</max_step_size>
@@ -7,9 +8,19 @@
     <gravity>0 0 -9.8</gravity>
   </physics>
+  <ros2_control name="GazeboSystem" type="system">
+    <hardware>
+        <plugin>gazebo_ros2_control/GazeboSystem</plugin>
+    </hardware>
+    <xacro:wheel_transmission side="lf_"/>
+    <xacro:wheel_transmission side="rf_"/>
+    <xacro:wheel_transmission side="rr_"/>
+    <xacro:wheel_transmission side="lr_"/>
+  </ros2_control>
   <gazebo>
-    <plugin name="gazebo_ros_control" filename="libgazebo_ros_control.so">
+    <plugin filename="libgazebo_ros2_control.so" name="gazebo_ros2_control">
       <robotNamespace></robotNamespace>
-      <robotSimType>gazebo_ros_control/DefaultRobotHWSim</robotSimType>
-      <legacyModeNS>true</legacyModeNS>
+      <robot_param>robot_description</robot_param>
+      <robot_param_node>robot_state_publisher</robot_param_node>
+      <parameters>$(find swerve_drive_description)/config/ros_controllers.yaml</parameters>
     </plugin>
   </gazebo>

File: swerve_drive_description/urdf/swerve_drive.xacro (robot description, xacro)
@@ -33,5 +33,5 @@
       <geometry>
         <mesh
-          filename="package://swerve_drive_description/meshes/base_link.STL" />
+          filename="file://$(find swerve_drive_description)/meshes/base_link.STL" />
       </geometry>
       <material
@@ -47,5 +47,5 @@
       <geometry>
         <mesh
-          filename="package://swerve_drive_description/meshes/base_link.STL" />
+          filename="file://$(find swerve_drive_description)/meshes/base_link.STL" />
       </geometry>
     </collision>

File: swerve_drive_description/urdf/wheel.transmission.xacro (robot description, xacro)
@@ -3,25 +3,18 @@
   <!-- parses the transmission tags and loads the appropriate hardware interfaces and controller manager -->
   <xacro:macro name="wheel_transmission" params="side">
-    <!-- all joint transmission -->
-    <transmission name="${side}swerve_joint_trans">
-        <type>transmission_interface/SimpleTransmission</type>
-        <joint name="${side}swerve_joint">
-            <hardwareInterface>hardware_interface/PositionJointInterface</hardwareInterface>
-        </joint>
-        <actuator name="${side}swerve_joint_motor">
-            <hardwareInterface>hardware_interface/PositionJointInterface</hardwareInterface>
-            <mechanicalReduction>1</mechanicalReduction>
-        </actuator>
-    </transmission>
-    <transmission name="${side}wheel_joint_trans">
-        <type>transmission_interface/SimpleTransmission</type>
-        <joint name="${side}wheel_joint">
-            <hardwareInterface>hardware_interface/VelocityJointInterface</hardwareInterface>
-        </joint>
-        <actuator name="${side}wheel_joint_motor">
-            <hardwareInterface>hardware_interface/VelocityJointInterface</hardwareInterface>
-            <mechanicalReduction>1</mechanicalReduction>
-        </actuator>
-    </transmission>
+    <joint name="${side}swerve_joint">
+        <command_interface name="position">
+        </command_interface>
+        <state_interface name="position"/>
+        <state_interface name="velocity"/>
+    </joint>
+    <joint name="${side}wheel_joint">
+        <command_interface name="velocity">
+            <param name="min">-1</param>
+            <param name="max">1</param>
+        </command_interface>
+        <state_interface name="position"/>
+        <state_interface name="velocity"/>
+    </joint>
   </xacro:macro>
 </robot>

File: swerve_drive_description/urdf/wheel.xacro (robot description, xacro)
@@ -2,5 +2,4 @@
 <robot xmlns:xacro="http://www.ros.org/wiki/xacro">
   <xacro:include filename="$(find swerve_drive_description)/urdf/wheel.gazebo.xacro" />
-  <xacro:include filename="$(find swerve_drive_description)/urdf/wheel.transmission.xacro" />
   <xacro:macro name="swerve_wheel" params="side parent *origin">
     <link
@@ -26,5 +25,5 @@
         <geometry>
             <mesh
-            filename="package://swerve_drive_description/meshes/swerve_link.STL" />
+                filename="file://$(find swerve_drive_description)/meshes/swerve_link.STL" />
         </geometry>
         <material
@@ -40,5 +39,5 @@
         <geometry>
             <mesh
-            filename="package://swerve_drive_description/meshes/swerve_link.STL" />
+                filename="file://$(find swerve_drive_description)/meshes/swerve_link.STL" />
         </geometry>
         </collision>
@@ -80,5 +79,5 @@
         <geometry>
             <mesh
-            filename="package://swerve_drive_description/meshes/wheel_link.STL" />
+                filename="file://$(find swerve_drive_description)/meshes/wheel_link.STL" />
         </geometry>
         <material
@@ -94,5 +93,5 @@
         <geometry>
             <mesh
-            filename="package://swerve_drive_description/meshes/wheel_link.STL" />
+                filename="file://$(find swerve_drive_description)/meshes/wheel_link.STL" />
         </geometry>
         </collision>
@@ -114,5 +113,4 @@
             velocity="12.7" />
     </joint>
-    <xacro:wheel_transmission side="${side}"/>
     <xacro:wheel_gazebo side="${side}"/>
   </xacro:macro>

Commit message: joy control without motion plan

File: swerve_drive_description/urdf/swerve_drive.gazebo.xacro (robot description, xacro)
@@ -1,5 +1,4 @@
 <?xml version="1.0"?>
 <robot name="swerve_drive" xmlns:xacro="http://www.ros.org/wiki/xacro">
-  <xacro:include filename="$(find swerve_drive_description)/urdf/wheel.transmission.xacro" />
   <physics type='ode'>
     <max_step_size>0.001</max_step_size>
@@ -8,21 +7,4 @@
     <gravity>0 0 -9.8</gravity>
   </physics>
-  <ros2_control name="GazeboSystem" type="system">
-    <hardware>
-        <plugin>gazebo_ros2_control/GazeboSystem</plugin>
-    </hardware>
-    <xacro:wheel_transmission side="lf_"/>
-    <xacro:wheel_transmission side="rf_"/>
-    <xacro:wheel_transmission side="rr_"/>
-    <xacro:wheel_transmission side="lr_"/>
-  </ros2_control>
-  <gazebo>
-    <plugin filename="libgazebo_ros2_control.so" name="gazebo_ros2_control">
-      <robotNamespace></robotNamespace>
-      <robot_param>robot_description</robot_param>
-      <robot_param_node>robot_state_publisher</robot_param_node>
-      <parameters>$(find swerve_drive_description)/config/ros_controllers.yaml</parameters>
-    </plugin>
-  </gazebo>
   <gazebo reference="base_link">
     <mu1>0.2</mu1>
@@ -31,3 +13,9 @@
     <selfCollide>false</selfCollide>
   </gazebo>
+  <gazebo>
+    <plugin filename="libgazebo_ros2_control.so" name="gazebo_ros2_control">
+      <robot_param>robot_description</robot_param>
+      <parameters>$(find swerve_drive_description)/config/ros_controllers.yaml</parameters>
+    </plugin>
+  </gazebo>
 </robot>

File: swerve_drive_description/urdf/swerve_drive.xacro (robot description, xacro)
@@ -3,4 +3,5 @@
   <xacro:include filename="$(find swerve_drive_description)/urdf/wheel.xacro" />
   <xacro:include filename="$(find swerve_drive_description)/urdf/swerve_drive.gazebo.xacro" />
+  <xacro:include filename="$(find swerve_drive_description)/urdf/swerve_drive.ros2_control.xacro" />
   <xacro:arg name="robot_type" default=""/>
   <xacro:arg name="name" default="" />
@@ -64,19 +65,17 @@
     </collision>
   </link>
-  <xacro:property name="lfj" value="${joints_info['lf']}" />
-  <xacro:property name="rfj" value="${joints_info['rf']}" />
-  <xacro:property name="rrj" value="${joints_info['rr']}" />
-  <xacro:property name="lrj" value="${joints_info['lr']}" />
+  <xacro:property name="swerve_joint" value="${joints_info['swerve']}" />
+  <xacro:property name="wheel_joint" value="${joints_info['wheel']}" />
   <xacro:swerve_wheel
-    side="lf_"  parent="base_link" mesh_files="${mesh_files}" swerve_joint="${lfj}"
-    wheel_joint="${joints_info['wheel']}" links="${links_info}" />
+    side="lf_"  parent="base_link" mesh_files="${mesh_files}" swerve_joint="${swerve_joint['lf']}"
+    wheel_joint="${wheel_joint['lf']}" links="${links_info}" />
   <xacro:swerve_wheel
-    side="rf_"  parent="base_link" mesh_files="${mesh_files}" swerve_joint="${rfj}"
-    wheel_joint="${joints_info['wheel']}" links="${links_info}" />
+    side="rf_"  parent="base_link" mesh_files="${mesh_files}" swerve_joint="${swerve_joint['rf']}"
+    wheel_joint="${wheel_joint['rf']}" links="${links_info}" />
   <xacro:swerve_wheel
-    side="rr_"  parent="base_link" mesh_files="${mesh_files}" swerve_joint="${rrj}"
-    wheel_joint="${joints_info['wheel']}" links="${links_info}" />
+    side="rr_"  parent="base_link" mesh_files="${mesh_files}" swerve_joint="${swerve_joint['rr']}"
+    wheel_joint="${wheel_joint['rr']}" links="${links_info}" />
   <xacro:swerve_wheel
-    side="lr_"  parent="base_link" mesh_files="${mesh_files}" swerve_joint="${lrj}"
-    wheel_joint="${joints_info['wheel']}" links="${links_info}" />
+    side="lr_"  parent="base_link" mesh_files="${mesh_files}" swerve_joint="${swerve_joint['lr']}"
+    wheel_joint="${wheel_joint['lr']}" links="${links_info}" />
 </robot>

File: swerve_drive_description/urdf/wheel.gazebo.xacro (robot description, xacro)
@@ -9,8 +9,8 @@
     </gazebo>
     <gazebo reference="${side}wheel_link">
-      <mu1 value="1.0"/>
-      <mu2 value="1.0"/>
-      <kp value="10000000.0" />
-      <kd value="1.0" />
+      <mu1 value="10.0"/>
+      <mu2 value="10.0"/>
+      <kp value="100000000.0" />
+      <kd value="10.0" />
       <fdir1 value="1 0 0"/>
       <material>Gazebo/Blue</material>

File: swerve_drive_description/urdf/wheel.ros2_control.xacro (robot description, xacro)
@@ -2,5 +2,5 @@
 <robot xmlns:xacro="http://www.ros.org/wiki/xacro">
   <!-- parses the transmission tags and loads the appropriate hardware interfaces and controller manager -->
-  <xacro:macro name="wheel_transmission" params="side">
+  <xacro:macro name="wheel_ros2_control" params="side swerve_id wheel_id">
     <joint name="${side}swerve_joint">
         <command_interface name="position">
@@ -8,12 +8,16 @@
         <state_interface name="position"/>
         <state_interface name="velocity"/>
+        <param name="motor_id">${swerve_id}</param>
+        <param name="mechanical_reduction">1</param>
     </joint>
     <joint name="${side}wheel_joint">
         <command_interface name="velocity">
-            <param name="min">-1</param>
-            <param name="max">1</param>
+            <param name="min">0</param>
+            <param name="max">0</param>
         </command_interface>
         <state_interface name="position"/>
         <state_interface name="velocity"/>
+        <param name="motor_id">${wheel_id}</param>
+        <param name="mechanical_reduction">1</param>
     </joint>
   </xacro:macro>

Commit message: replace collision mesh

File: swerve_drive_description/urdf/swerve_drive.gazebo.xacro (robot description, xacro)
@@ -10,5 +10,5 @@
     <mu1>0.2</mu1>
     <mu2>0.2</mu2>
-    <material>Gazebo/Gray</material>
+    <material>Gazebo/White</material>
     <selfCollide>false</selfCollide>
   </gazebo>

File: swerve_drive_description/urdf/swerve_drive.xacro (robot description, xacro)
@@ -7,13 +7,15 @@
   <xacro:arg name="name" default="" />
   <xacro:arg name="prefix" default="" />
-  <xacro:arg name="visual_parameters_file" default="$(find swerve_drive_description)/config/$(arg robot_type)/visual_parameters.yaml" />
+  <xacro:arg name="geometry_parameters_file" default="$(find swerve_drive_description)/config/$(arg robot_type)/geometry_parameters.yaml" />
   <xacro:arg name="physical_parameters_file" default="$(find swerve_drive_description)/config/$(arg robot_type)/physical_parameters.yaml" />
-  <xacro:property name="config_visual_parameters" value="${load_yaml('$(arg visual_parameters_file)')}" />
+  <xacro:property name="config_geometry_parameters" value="${load_yaml('$(arg geometry_parameters_file)')}" />
   <xacro:property name="config_physical_parameters" value="${load_yaml('$(arg physical_parameters_file)')}" />
-  <xacro:property name="mesh_files" value="${config_visual_parameters['mesh_files']}" />
+  <xacro:property name="geometry_config" value="${config_geometry_parameters['geometry_config']}" />
   <xacro:property name="joints_info" value="${config_physical_parameters['joints']}" />
   <xacro:property name="links_info" value="${config_physical_parameters['links']}" />
   <xacro:property name="bio" value="${links_info['base']['inertial']['origin']}" />
   <xacro:property name="bii" value="${links_info['base']['inertial']['inertia']}" />
+  <xacro:property name="bvo" value="${geometry_config['base']['visual']['origin']}" />
+  <xacro:property name="bco" value="${geometry_config['base']['collision']['origin']}" />
   <xacro:property name="jbo" value="${joints_info['base']['origin']}" />
   <link name="base_footprint"/>
@@ -43,9 +45,9 @@
     <visual>
       <origin
-        xyz="0 0 0"
-        rpy="0 0 0" />
+        xyz="${bvo['x']} ${bvo['y']} ${bvo['z']}"
+        rpy="${bvo['roll']} ${bvo['pitch']} ${bvo['yaw']}" />
       <geometry>
         <mesh
-          filename="file://$(find ${mesh_files['package']})/${mesh_files['base']['visual']['path']}" />
+          filename="file://$(find ${geometry_config['package']})/${geometry_config['base']['visual']['path']}" />
       </geometry>
       <material
@@ -57,9 +59,9 @@
     <collision>
       <origin
-        xyz="0 0 0"
-        rpy="0 0 0" />
+        xyz="${bco['x']} ${bco['y']} ${bco['z']}"
+        rpy="${bco['roll']} ${bco['pitch']} ${bco['yaw']}" />
       <geometry>
         <mesh
-          filename="file://$(find ${mesh_files['package']})/${mesh_files['base']['collision']['path']}" />
+          filename="file://$(find ${geometry_config['package']})/${geometry_config['base']['collision']['path']}" />
       </geometry>
     </collision>
@@ -68,14 +70,14 @@
   <xacro:property name="wheel_joint" value="${joints_info['wheel']}" />
   <xacro:swerve_wheel
-    side="lf_"  parent="base_link" mesh_files="${mesh_files}" swerve_joint="${swerve_joint['lf']}"
+    side="lf_"  parent="base_link" geometry_config="${geometry_config}" swerve_joint="${swerve_joint['lf']}"
     wheel_joint="${wheel_joint['lf']}" links="${links_info}" />
   <xacro:swerve_wheel
-    side="rf_"  parent="base_link" mesh_files="${mesh_files}" swerve_joint="${swerve_joint['rf']}"
+    side="rf_"  parent="base_link" geometry_config="${geometry_config}" swerve_joint="${swerve_joint['rf']}"
     wheel_joint="${wheel_joint['rf']}" links="${links_info}" />
   <xacro:swerve_wheel
-    side="rr_"  parent="base_link" mesh_files="${mesh_files}" swerve_joint="${swerve_joint['rr']}"
+    side="rr_"  parent="base_link" geometry_config="${geometry_config}" swerve_joint="${swerve_joint['rr']}"
     wheel_joint="${wheel_joint['rr']}" links="${links_info}" />
   <xacro:swerve_wheel
-    side="lr_"  parent="base_link" mesh_files="${mesh_files}" swerve_joint="${swerve_joint['lr']}"
+    side="lr_"  parent="base_link" geometry_config="${geometry_config}" swerve_joint="${swerve_joint['lr']}"
     wheel_joint="${wheel_joint['lr']}" links="${links_info}" />
 </robot>

File: swerve_drive_description/urdf/wheel.xacro (robot description, xacro)
@@ -2,5 +2,5 @@
 <robot xmlns:xacro="http://www.ros.org/wiki/xacro">
   <xacro:include filename="$(find swerve_drive_description)/urdf/wheel.gazebo.xacro" />
-  <xacro:macro name="swerve_wheel" params="side parent  mesh_files swerve_joint wheel_joint links">
+  <xacro:macro name="swerve_wheel" params="side parent geometry_config swerve_joint wheel_joint links">
     <xacro:property name="sjo" value="${swerve_joint['origin']}" />
     <xacro:property name="sja" value="${swerve_joint['axis']}" />
@@ -11,4 +11,8 @@
     <xacro:property name="wio" value="${links['wheel']['inertial']['origin']}" />
     <xacro:property name="wii" value="${links['wheel']['inertial']['inertia']}" />
+    <xacro:property name="svo" value="${geometry_config['swerve']['visual']['origin']}" />
+    <xacro:property name="sco" value="${geometry_config['swerve']['collision']['origin']}" />
+    <xacro:property name="wvo" value="${geometry_config['wheel']['visual']['origin']}" />
+    <xacro:property name="wco" value="${geometry_config['wheel']['collision']['origin']}" />
     <link
         name="${side}swerve_link">
@@ -29,9 +33,9 @@
         <visual>
             <origin
-                xyz="0 0 0"
-                rpy="0 0 0" />
+                xyz="${svo['x']} ${svo['y']} ${svo['z']}"
+                rpy="${svo['roll']} ${svo['pitch']} ${svo['yaw']}" />
             <geometry>
                 <mesh
-                    filename="file://$(find ${mesh_files['package']})/${mesh_files['swerve']['visual']['path']}" />
+                    filename="file://$(find ${geometry_config['package']})/${geometry_config['swerve']['visual']['path']}" />
             </geometry>
             <material
@@ -43,9 +47,9 @@
         <collision>
             <origin
-                xyz="0 0 0"
-                rpy="0 0 0" />
+                xyz="${sco['x']} ${sco['y']} ${sco['z']}"
+                rpy="${sco['roll']} ${sco['pitch']} ${sco['yaw']}" />
             <geometry>
                 <mesh
-                    filename="file://$(find ${mesh_files['package']})/${mesh_files['swerve']['collision']['path']}" />
+                    filename="file://$(find ${geometry_config['package']})/${geometry_config['swerve']['collision']['path']}" />
             </geometry>
         </collision>
@@ -85,9 +89,9 @@
         <visual>
             <origin
-                xyz="0 0 0"
-                rpy="0 0 0" />
+                xyz="${wco['x']} ${wco['y']} ${wco['z']}"
+                rpy="${wco['roll']} ${wco['pitch']} ${wco['yaw']}" />
             <geometry>
                 <mesh
-                    filename="file://$(find ${mesh_files['package']})/${mesh_files['wheel']['visual']['path']}" />
+                    filename="file://$(find ${geometry_config['package']})/${geometry_config['wheel']['visual']['path']}" />
             </geometry>
             <material
@@ -99,9 +103,9 @@
         <collision>
             <origin
-                xyz="0 0 0"
-                rpy="0 0 0" />
+                xyz="${wvo['x']} ${wvo['y']} ${wvo['z']}"
+                rpy="${wvo['roll']} ${wvo['pitch']} ${wvo['yaw']}" />
             <geometry>
                 <mesh
-                    filename="file://$(find ${mesh_files['package']})/${mesh_files['wheel']['collision']['path']}" />
+                    filename="file://$(find ${geometry_config['package']})/${geometry_config['wheel']['collision']['path']}" />
             </geometry>
         </collision>
