Commit message: make xacro easier to be include

File: swerve_drive_description/urdf/swerve_drive.gazebo.xacro (robot description, xacro)
@@ -1,21 +1,11 @@
 <?xml version="1.0"?>
-<robot name="swerve_drive" xmlns:xacro="http://www.ros.org/wiki/xacro">
-  <physics type='ode'>
-    <max_step_size>0.001</max_step_size>
-    <real_time_factor>0.1</real_time_factor>
-    <real_time_update_rate>1000</real_time_update_rate>
-    <gravity>0 0 -9.8</gravity>
-  </physics>
-  <gazebo reference="base_link">
-    <mu1>0.2</mu1>
-    <mu2>0.2</mu2>
-    <material>Gazebo/White</material>
-    <selfCollide>false</selfCollide>
-  </gazebo>
-  <gazebo>
-    <plugin filename="libgazebo_ros2_control.so" name="gazebo_ros2_control">
-      <robot_param>robot_description</robot_param>
-      <parameters>$(find swerve_drive_description)/config/ros_controllers.yaml</parameters>
-    </plugin>
-  </gazebo>
+<robot xmlns:xacro="http://www.ros.org/wiki/xacro">
+  <xacro:macro name="swerve_drive_gazebo" params="prefix">
+    <gazebo reference="${prefix}base_link">
+      <mu1>0.2</mu1>
+      <mu2>0.2</mu2>
+      <material>Gazebo/White</material>
+      <selfCollide>false</selfCollide>
+    </gazebo>
+  </xacro:macro>
 </robot>

File: swerve_drive_description/urdf/swerve_drive.ros2_control.xacro (robot description, xacro)
@@ -2,12 +2,26 @@
 <robot name="swerve_drive" xmlns:xacro="http://www.ros.org/wiki/xacro">
   <xacro:include filename="$(find swerve_drive_description)/urdf/wheel.ros2_control.xacro" />
-  <ros2_control name="GazeboSystem" type="system">
-    <hardware>
-        <plugin>gazebo_ros2_control/GazeboSystem</plugin>
-    </hardware>
-    <xacro:wheel_ros2_control side="lf_" swerve_id="0" wheel_id="1"/>
-    <xacro:wheel_ros2_control side="rf_" swerve_id="2" wheel_id="3"/>
-    <xacro:wheel_ros2_control side="rr_" swerve_id="4" wheel_id="5"/>
-    <xacro:wheel_ros2_control side="lr_" swerve_id="6" wheel_id="7"/>
-  </ros2_control>
+  <xacro:macro name="swerve_drive_ros2_control" params="prefix">
+    <physics type='ode'>
+      <max_step_size>0.001</max_step_size>
+      <real_time_factor>0.1</real_time_factor>
+      <real_time_update_rate>1000</real_time_update_rate>
+      <gravity>0 0 -9.8</gravity>
+    </physics>
+    <gazebo>
+      <plugin filename="libgazebo_ros2_control.so" name="gazebo_ros2_control">
+        <robot_param>robot_description</robot_param>
+        <parameters>$(find swerve_drive_description)/config/ros_controllers.yaml</parameters>
+      </plugin>
+    </gazebo>
+    <ros2_control name="GazeboSystem" type="system">
+      <hardware>
+          <plugin>gazebo_ros2_control/GazeboSystem</plugin>
+      </hardware>
+      <xacro:wheel_ros2_control prefix="${prefix}" side="lf_" swerve_id="0" wheel_id="1"/>
+      <xacro:wheel_ros2_control prefix="${prefix}" side="rf_" swerve_id="2" wheel_id="3"/>
+      <xacro:wheel_ros2_control prefix="${prefix}" side="rr_" swerve_id="4" wheel_id="5"/>
+      <xacro:wheel_ros2_control prefix="${prefix}" side="lr_" swerve_id="6" wheel_id="7"/>
+    </ros2_control>
+  </xacro:macro>
 </robot>

File: swerve_drive_description/urdf/swerve_drive.xacro (robot description, xacro)
@@ -1,83 +1,84 @@
 <?xml version="1.0"?>
-<robot name="$(arg name)" xmlns:xacro="http://www.ros.org/wiki/xacro">
+<robot xmlns:xacro="http://www.ros.org/wiki/xacro">
   <xacro:include filename="$(find swerve_drive_description)/urdf/wheel.xacro" />
   <xacro:include filename="$(find swerve_drive_description)/urdf/swerve_drive.gazebo.xacro" />
-  <xacro:include filename="$(find swerve_drive_description)/urdf/swerve_drive.ros2_control.xacro" />
-  <xacro:arg name="robot_type" default=""/>
-  <xacro:arg name="name" default="" />
-  <xacro:arg name="prefix" default="" />
-  <xacro:arg name="geometry_parameters_file" default="$(find swerve_drive_description)/config/$(arg robot_type)/geometry_parameters.yaml" />
-  <xacro:arg name="physical_parameters_file" default="$(find swerve_drive_description)/config/$(arg robot_type)/physical_parameters.yaml" />
-  <xacro:property name="config_geometry_parameters" value="${load_yaml('$(arg geometry_parameters_file)')}" />
-  <xacro:property name="config_physical_parameters" value="${load_yaml('$(arg physical_parameters_file)')}" />
-  <xacro:property name="geometry_config" value="${config_geometry_parameters['geometry_config']}" />
-  <xacro:property name="joints_info" value="${config_physical_parameters['joints']}" />
-  <xacro:property name="links_info" value="${config_physical_parameters['links']}" />
-  <xacro:property name="bio" value="${links_info['base']['inertial']['origin']}" />
-  <xacro:property name="bii" value="${links_info['base']['inertial']['inertia']}" />
-  <xacro:property name="bvo" value="${geometry_config['base']['visual']['origin']}" />
-  <xacro:property name="bco" value="${geometry_config['base']['collision']['origin']}" />
-  <xacro:property name="jbo" value="${joints_info['base']['origin']}" />
-  <link name="base_footprint"/>
-  <joint name="base_joint " type="fixed">
-    <origin
-      xyz="${jbo['x']} ${jbo['y']} ${jbo['z']}"
-      rpy="${jbo['roll']} ${jbo['pitch']} ${jbo['yaw']}" />
-    <parent link="base_footprint"/>
-    <child link="base_link"/>
-  </joint>
-  <link
-    name="base_link">
-    <inertial>
+  <!-- <xacro:arg name="robot_type" default=""/> -->
+  <!-- <xacro:arg name="name" default="" /> -->
+  <!-- <xacro:arg name="prefix" default="" /> -->
+  <!-- <xacro:arg name="geometry_parameters_file" default="$(find swerve_drive_description)/config/$(arg robot_type)/geometry_parameters.yaml" /> -->
+  <!-- <xacro:arg name="physical_parameters_file" default="$(find swerve_drive_description)/config/$(arg robot_type)/physical_parameters.yaml" /> -->
+  <xacro:macro name="swerve_drive" params="name robot_type prefix parent geometry_parameters_file physical_parameters_file">
+    <xacro:property name="config_geometry_parameters" value="${load_yaml(geometry_parameters_file)}" />
+    <xacro:property name="config_physical_parameters" value="${load_yaml(physical_parameters_file)}" />
+    <xacro:property name="geometry_config" value="${config_geometry_parameters['geometry_config']}" />
+    <xacro:property name="joints_info" value="${config_physical_parameters['joints']}" />
+    <xacro:property name="links_info" value="${config_physical_parameters['links']}" />
+    <xacro:property name="bio" value="${links_info['base']['inertial']['origin']}" />
+    <xacro:property name="bii" value="${links_info['base']['inertial']['inertia']}" />
+    <xacro:property name="bvo" value="${geometry_config['base']['visual']['origin']}" />
+    <xacro:property name="bco" value="${geometry_config['base']['collision']['origin']}" />
+    <xacro:property name="jbo" value="${joints_info['base']['origin']}" />
+    <joint name="${prefix}base_joint " type="fixed">
       <origin
-        xyz="${bio['x']} ${bio['y']} ${bio['z']}"
-        rpy="${bio['roll']} ${bio['pitch']} ${bio['yaw']}" />
-      <mass
-        value="${links_info['base']['inertial']['mass']}" />
-      <inertia
-        ixx="${bii['xx']}"
-        ixy="0"
-        ixz="0"
-        iyy="${bii['yy']}"
-        iyz="0"
-        izz="${bii['zz']}" />
-    </inertial>
-    <visual>
-      <origin
-        xyz="${bvo['x']} ${bvo['y']} ${bvo['z']}"
-        rpy="${bvo['roll']} ${bvo['pitch']} ${bvo['yaw']}" />
-      <geometry>
-        <mesh
-          filename="file://$(find ${geometry_config['package']})/${geometry_config['base']['visual']['path']}" />
-      </geometry>
-      <material
-        name="">
-        <color
-          rgba="0.75294 0.75294 0.75294 1" />
-      </material>
-    </visual>
-    <collision>
-      <origin
-        xyz="${bco['x']} ${bco['y']} ${bco['z']}"
-        rpy="${bco['roll']} ${bco['pitch']} ${bco['yaw']}" />
-      <geometry>
-        <mesh
-          filename="file://$(find ${geometry_config['package']})/${geometry_config['base']['collision']['path']}" />
-      </geometry>
-    </collision>
-  </link>
-  <xacro:property name="swerve_joint" value="${joints_info['swerve']}" />
-  <xacro:property name="wheel_joint" value="${joints_info['wheel']}" />
-  <xacro:swerve_wheel
-    side="lf_"  parent="base_link" geometry_config="${geometry_config}" swerve_joint="${swerve_joint['lf']}"
-    wheel_joint="${wheel_joint['lf']}" links="${links_info}" />
-  <xacro:swerve_wheel
-    side="rf_"  parent="base_link" geometry_config="${geometry_config}" swerve_joint="${swerve_joint['rf']}"
-    wheel_joint="${wheel_joint['rf']}" links="${links_info}" />
-  <xacro:swerve_wheel
-    side="rr_"  parent="base_link" geometry_config="${geometry_config}" swerve_joint="${swerve_joint['rr']}"
-    wheel_joint="${wheel_joint['rr']}" links="${links_info}" />
-  <xacro:swerve_wheel
-    side="lr_"  parent="base_link" geometry_config="${geometry_config}" swerve_joint="${swerve_joint['lr']}"
-    wheel_joint="${wheel_joint['lr']}" links="${links_info}" />
+        xyz="${jbo['x']} ${jbo['y']} ${jbo['z']}"
+        rpy="${jbo['roll']} ${jbo['pitch']} ${jbo['yaw']}" />
+      <parent link="${parent}"/>
+      <child link="${prefix}base_link"/>
+    </joint>
+    <link
+      name="${prefix}base_link">
+      <inertial>
+        <origin
+          xyz="${bio['x']} ${bio['y']} ${bio['z']}"
+          rpy="${bio['roll']} ${bio['pitch']} ${bio['yaw']}" />
+        <mass
+          value="${links_info['base']['inertial']['mass']}" />
+        <inertia
+          ixx="${bii['xx']}"
+          ixy="0"
+          ixz="0"
+          iyy="${bii['yy']}"
+          iyz="0"
+          izz="${bii['zz']}" />
+      </inertial>
+      <visual>
+        <origin
+          xyz="${bvo['x']} ${bvo['y']} ${bvo['z']}"
+          rpy="${bvo['roll']} ${bvo['pitch']} ${bvo['yaw']}" />
+        <geometry>
+          <mesh
+            filename="file://$(find ${geometry_config['package']})/${geometry_config['base']['visual']['path']}" />
+        </geometry>
+        <material
+          name="">
+          <color
+            rgba="0.75294 0.75294 0.75294 1" />
+        </material>
+      </visual>
+      <collision>
+        <origin
+          xyz="${bco['x']} ${bco['y']} ${bco['z']}"
+          rpy="${bco['roll']} ${bco['pitch']} ${bco['yaw']}" />
+        <geometry>
+          <mesh
+            filename="file://$(find ${geometry_config['package']})/${geometry_config['base']['collision']['path']}" />
+        </geometry>
+      </collision>
+    </link>
+    <xacro:property name="swerve_joint" value="${joints_info['swerve']}" />
+    <xacro:property name="wheel_joint" value="${joints_info['wheel']}" />
+    <xacro:swerve_wheel
+      side="lf_"  parent="${prefix}base_link" prefix="${prefix}" geometry_config="${geometry_config}"
+      swerve_joint="${swerve_joint['lf']}" wheel_joint="${wheel_joint['lf']}" links="${links_info}" />
+    <xacro:swerve_wheel
+      side="rf_"  parent="${prefix}base_link" prefix="${prefix}" geometry_config="${geometry_config}"
+      swerve_joint="${swerve_joint['rf']}" wheel_joint="${wheel_joint['rf']}" links="${links_info}" />
+    <xacro:swerve_wheel
+      side="rr_"  parent="${prefix}base_link" prefix="${prefix}" geometry_config="${geometry_config}"
+      swerve_joint="${swerve_joint['rr']}" wheel_joint="${wheel_joint['rr']}" links="${links_info}" />
+    <xacro:swerve_wheel
+      side="lr_"  parent="${prefix}base_link" prefix="${prefix}" geometry_config="${geometry_config}"
+      swerve_joint="${swerve_joint['lr']}" wheel_joint="${wheel_joint['lr']}" links="${links_info}" />
+    <xacro:swerve_drive_gazebo prefix="${prefix}"/>
+  </xacro:macro>
 </robot>

File: swerve_drive_description/urdf/wheel.gazebo.xacro (robot description, xacro)
@@ -1,6 +1,6 @@
 <?xml version="1.0"?>
 <robot xmlns:xacro="http://www.ros.org/wiki/xacro">
-  <xacro:macro name="wheel_gazebo" params="side">
-    <gazebo reference="${side}swerve_link">
+  <xacro:macro name="wheel_gazebo" params="side prefix">
+    <gazebo reference="${prefix}${side}swerve_link">
       <mu1 value="0.1"/>
       <mu2 value="0.1"/>
@@ -8,5 +8,5 @@
       <selfCollide>false</selfCollide>
     </gazebo>
-    <gazebo reference="${side}wheel_link">
+    <gazebo reference="${prefix}${side}wheel_link">
       <mu1 value="10.0"/>
       <mu2 value="10.0"/>
@@ -17,8 +17,8 @@
       <selfCollide>false</selfCollide>
     </gazebo>
-    <gazebo reference="${side}swerve_joint">
+    <gazebo reference="${prefix}${side}swerve_joint">
       <implicitSpringDamper>True</implicitSpringDamper>
     </gazebo>
-    <gazebo reference="${side}wheel_joint">
+    <gazebo reference="${prefix}${side}wheel_joint">
       <implicitSpringDamper>True</implicitSpringDamper>
     </gazebo>

File: swerve_drive_description/urdf/wheel.ros2_control.xacro (robot description, xacro)
@@ -2,6 +2,6 @@
 <robot xmlns:xacro="http://www.ros.org/wiki/xacro">
   <!-- parses the transmission tags and loads the appropriate hardware interfaces and controller manager -->
-  <xacro:macro name="wheel_ros2_control" params="side swerve_id wheel_id">
-    <joint name="${side}swerve_joint">
+  <xacro:macro name="wheel_ros2_control" params="side prefix swerve_id wheel_id">
+    <joint name="${prefix}${side}swerve_joint">
         <command_interface name="position">
         </command_interface>
@@ -11,5 +11,5 @@
         <param name="mechanical_reduction">1</param>
     </joint>
-    <joint name="${side}wheel_joint">
+    <joint name="${prefix}${side}wheel_joint">
         <command_interface name="velocity">
             <param name="min">0</param>

File: swerve_drive_description/urdf/wheel.xacro (robot description, xacro)
@@ -2,5 +2,5 @@
 <robot xmlns:xacro="http://www.ros.org/wiki/xacro">
   <xacro:include filename="$(find swerve_drive_description)/urdf/wheel.gazebo.xacro" />
-  <xacro:macro name="swerve_wheel" params="side parent geometry_config swerve_joint wheel_joint links">
+  <xacro:macro name="swerve_wheel" params="prefix side parent geometry_config swerve_joint wheel_joint links">
     <xacro:property name="sjo" value="${swerve_joint['origin']}" />
     <xacro:property name="sja" value="${swerve_joint['axis']}" />
@@ -16,5 +16,5 @@
     <xacro:property name="wco" value="${geometry_config['wheel']['collision']['origin']}" />
     <link
-        name="${side}swerve_link">
+        name="${prefix}${side}swerve_link">
         <inertial>
             <origin
@@ -56,5 +56,5 @@
     </link>
     <joint
-        name="${side}swerve_joint"
+        name="${prefix}${side}swerve_joint"
         type="continuous">
         <origin
@@ -64,5 +64,5 @@
             link="${parent}" />
         <child
-            link="${side}swerve_link" />
+            link="${prefix}${side}swerve_link" />
         <axis
             xyz="${sja['x']} ${sja['y']} ${sja['z']}" />
@@ -72,5 +72,5 @@
     </joint>
     <link
-        name="${side}wheel_link">
+        name="${prefix}${side}wheel_link">
         <inertial>
             <origin
@@ -112,5 +112,5 @@
     </link>
     <joint
-        name="${side}wheel_joint"
+        name="${prefix}${side}wheel_joint"
         type="continuous">
         <origin
@@ -118,7 +118,7 @@
             rpy="${wjo['roll']} ${wjo['pitch']} ${wjo['yaw']}" />
         <parent
-            link="${side}swerve_link" />
+            link="${prefix}${side}swerve_link" />
         <child
-            link="${side}wheel_link" />
+            link="${prefix}${side}wheel_link" />
         <axis
             xyz="${wja['x']} ${wja['y']} ${wja['z']}" />
@@ -127,5 +127,5 @@
             velocity="12.7" />
     </joint>
-    <xacro:wheel_gazebo side="${side}"/>
+    <xacro:wheel_gazebo side="${side}" prefix="${prefix}"/>
   </xacro:macro>
 </robot>
