Commit message: disable some useless params

File: swerve_drive_description/urdf/wheel.gazebo.xacro (robot description, xacro)
@@ -3,20 +3,20 @@
   <xacro:macro name="wheel_gazebo" params="side prefix">
     <gazebo reference="${prefix}${side}swerve_link">
-      <mu1 value="0.1"/>
-      <mu2 value="0.1"/>
+      <!-- <mu1 value="0.1"/> -->
+      <!-- <mu2 value="0.1"/> -->
       <material>Gazebo/Black</material>
       <selfCollide>false</selfCollide>
     </gazebo>
     <gazebo reference="${prefix}${side}wheel_link">
-      <mu value="100000.0"/>
-      <mu1 value="100000.0"/>
-      <mu2 value="100000.0"/>
-      <soft_cfm value="0" />
-      <soft_erp value="0.02" />
+      <!-- <mu value="100000.0"/> -->
+      <!-- <mu1 value="100000.0"/> -->
+      <!-- <mu2 value="100000.0"/> -->
+      <!-- <soft_cfm value="0" /> -->
+      <!-- <soft_erp value="0.02" /> -->
       <kp value="100000.0" />
       <kd value="10000000000000.0" />
-      <max_vel value="0.01" />
-      <min_vel value="0.001" />
-      <fdir1 value="0 0 0"/>
+      <!-- <max_vel value="0.01" /> -->
+      <!-- <min_vel value="0.001" /> -->
+      <!-- <fdir1 value="0 0 0"/> -->
       <material>Gazebo/Blue</material>
       <selfCollide>false</selfCollide>

File: swerve_drive_description/urdf/wheel.xacro (robot description, xacro)
@@ -70,7 +70,7 @@
             effort="100"
             velocity="3.2" />
-        <dynamics
+        <!-- <dynamics
             damping="100"
-            friction="10" />
+            friction="10" /> -->
     </joint>
     <link
@@ -129,7 +129,7 @@
             effort="30"
             velocity="12.7" />
-        <dynamics
+        <!-- <dynamics
             damping="0.4"
-            friction="0.04" />
+            friction="0.04" /> -->
     </joint>
     <xacro:wheel_gazebo side="${side}" prefix="${prefix}"/>
