Commit message: Simulater tested

File: swerve_drive_description/urdf/wheel.xacro (robot description, xacro)
@@ -49,9 +49,12 @@
         <xacro:insert_block name="origin" />
         <parent
-        link="${parent}" />
+            link="${parent}" />
         <child
-        link="${side}swerve_link" />
+            link="${side}swerve_link" />
         <axis
-        xyz="0 0 1" />
+            xyz="0 0 1" />
+        <limit
+            effort="100"
+            velocity="3.2" />
     </joint>
     <link
@@ -99,12 +102,15 @@
         type="continuous">
         <origin
-        xyz="0 0.00047482 -0.07"
-        rpy="0 0 0" />
+            xyz="0 0.00047482 -0.07"
+            rpy="0 0 0" />
         <parent
-        link="${side}swerve_link" />
+            link="${side}swerve_link" />
         <child
-        link="${side}wheel_link" />
+            link="${side}wheel_link" />
         <axis
-        xyz="0 1 0" />
+            xyz="0 1 0" />
+        <limit
+            effort="100"
+            velocity="12.7" />
     </joint>
     <xacro:wheel_transmission side="${side}"/>

Commit message: control in sim with mobile manipulator

File: swerve_drive_description/urdf/wheel.xacro (robot description, xacro)
@@ -70,4 +70,7 @@
             effort="100"
             velocity="3.2" />
+        <dynamics
+            damping="100"
+            friction="10" />
     </joint>
     <link
@@ -126,4 +129,7 @@
             effort="0.3"
             velocity="12.7" />
+        <dynamics
+            damping="40"
+            friction="4" />
     </joint>
     <xacro:wheel_gazebo side="${side}" prefix="${prefix}"/>

Commit message: visual link on wheel

File: swerve_drive_description/urdf/wheel.xacro (robot description, xacro)
@@ -133,4 +133,31 @@
             friction="0.04" /> -->
     </joint>
+    <link
+        name="${prefix}${side}wheel_arrow_link">
+        <visual>
+            <origin
+                xyz="0 0 0.05"
+                rpy="0 0 0" />
+            <geometry>
+                <box size="0.02 0.02 0.1" />
+            </geometry>
+            <material
+                name="">
+                <color
+                rgba="0.75294 0.75294 0.75294 1" />
+            </material>
+        </visual>
+    </link>
+    <joint
+        name="${prefix}${side}wheel_arrow_joint"
+        type="fixed">
+        <origin
+            xyz="0 -0.04 0"
+            rpy="0 0 0" />
+        <parent
+            link="${prefix}${side}wheel_link" />
+        <child
+            link="${prefix}${side}wheel_arrow_link" />
+    </joint>
     <xacro:wheel_gazebo side="${side}" prefix="${prefix}"/>
   </xacro:macro>
